File: paul_files/5V regulated power supply pcbdesign.kicad_pcb (KiCad board)
At the start: 2 copper layers, 67 x 61.6 mm, 14 parts, among them J1 AC_INPUT, J2 +10V, GND, T1 Transformer_1P_1S, U1 LM317

Commit message: changes_to_files
Parts:
- J2: value +10V, GND -> (+5v, gnd)
- R1: value 240 -> 150
- U1: value LM317 -> L7805
Other:
- board text added: "5V Regulated Power Supply"
- board text removed: "10V Regulated Power Supply"
Changed lines of the file:
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@@
 			)
 		)
-		(property "Value" "LM317 "
+		(property "Value" "L7805"
 			(at 2.54 2.2 0)
 			(layer "F.Fab")
@@
 			)
 		)
-		(property "Datasheet" ""
+		(property "Datasheet" "http://www.st.com/content/ccc/resource/technical/document/datasheet/41/4f/b3/b0/12/d4/47/88/CD00000444.pdf/files/CD00000444.pdf/jcr:content/translations/en.CD00000444.pdf"
 			(at 0 0 0)
 			(layer "F.Fab")
@@
 			)
 		)
-		(property "Description" ""
+		(property "Description" "Positive 1.5A 35V Linear Regulator, Fixed Output 5V, TO-220/TO-263/TO-252"
 			(at 0 0 0)
 			(layer "F.Fab")
@@
 			)
 		)
-		(property "Value" "+10V, GND "
+		(property "Value" "(+5v, gnd)"
 			(at 2.25 4.92 0)
 			(layer "F.Fab")
@@
 			)
 		)
-		(property "Value" "240"
+		(property "Value" "150"
 			(at 0.95 1.92 90)
 			(layer "F.Fab")
@@
 		(layer "Edge.Cuts")
 	)
-	(gr_text "10V Regulated Power Supply "
+	(gr_text "5V Regulated Power Supply "
 		(at 116.4 132.8 0)
 		(layer "F.SilkS")
