File: pcb_designs/S20240020331_Shounak_RPS_Diode_10V.kicad_pcb (KiCad board)
At the start: 2 copper layers, 67 x 61.6 mm, 14 parts, among them J1 AC_INPUT, J2 (+5v, gnd), T1 Transformer_1P_1S, U1 L7805

Commit message: major_fixes_to_ppl
Parts:
- J2: value (+5v, gnd) -> (+10v, gnd)
Other:
- board text added: "10V Regulated Power Supply"
- board text removed: "5V Regulated Power Supply"
Changed lines of the file:
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@@
 			)
 		)
-		(property "Value" "(+5v, gnd)"
+		(property "Value" "(+10v, gnd)"
 			(at 2.25 4.92 0)
 			(layer "F.Fab")
@@
 		(layer "Edge.Cuts")
 	)
-	(gr_text "5V Regulated Power Supply "
+	(gr_text "10V Regulated Power Supply "
 		(at 116.4 132.8 0)
 		(layer "F.SilkS")
